File: KAPTON-HEATERV2.kicad_pcb (KiCad board)
At the start: 2 copper layers, 90 x 75 mm, 19 parts, among them J1 XT60PW-M, J2 XT60PW-M, J3 1985276, J4 1985218, J5 10090926-P154XLF, K1 1-1393210-8, Q1 AO3400A, U1 TC4427ACOA

Commit message: added mounting holes
Parts:
- added REF**: MountingHole_2.2mm_M2, MountingHole:MountingHole_2.2mm_M2, F.Cu at (135.0, 130.0)
- added REF**: MountingHole_2.2mm_M2, MountingHole:MountingHole_2.2mm_M2, F.Cu at (135.0, 50.0)
- added REF**: MountingHole_2.2mm_M2, MountingHole:MountingHole_2.2mm_M2, F.Cu at (55.0, 50.0)
- added REF**: MountingHole_2.2mm_M2, MountingHole:MountingHole_2.2mm_M2, F.Cu at (55.0, 130.0)
- moved G*** 28.4 mm to (55.2, 112.7)
- moved C1 28.4 mm to (77.5, 70.5)
- moved C2 28.4 mm to (89.0, 71.0)
- moved C3 28.4 mm to (114.1, 71.5)
- moved C4 28.4 mm to (100.0, 69.5)
- moved D1 28.4 mm to (85.8, 63.5)
- moved F1 28.4 mm to (115.0, 115.0)
- moved J1 28.4 mm to (61.0, 97.5)
- moved J2 28.4 mm to (129.0, 116.2)
- moved J5 28.4 mm to (61.5, 69.0)
- moved K1 28.4 mm to (94.9, 103.4)
- moved MOSFET1 28.4 mm to (108.6, 70.9)
- moved Q1 28.4 mm to (83.5, 71.0)
- moved R1 28.4 mm to (121.5, 60.1)
- moved R2 28.4 mm to (121.5, 63.9)
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Routing:
- net TH8: track 92.2 -> 38.0 mm
- removed copper zone on B.Cu, net GND
Other:
- board size 90 x 75 mm -> 90 x 90 mm

Commit message: finalized?
Parts:
- removed C1: C0.1uf, Capacitor_SMD:C_0805_2012Metric
- removed C2: C47uf, Capacitor_THT:CP_Radial_D6.3mm_P2.50mm
- removed C3: C1uf, Capacitor_SMD:C_0805_2012Metric
- C4: value C10uf -> C47.5nf; footprint Capacitor_THT:CP_Radial_D6.3mm_P2.50mm -> Capacitor_SMD:C_0805_2012Metric
- moved C4 13.9 mm to (113.6, 72.2)
Connections:
- net /24VIN2 renamed Net-(F1-Pad2)
- J2 pad S1: GND -> (no net)
- J2 pad S2: GND -> (no net)
- J5 pad 10: unconnected-(J5-Pad10) -> 5V
- J5 pad 11: 5V -> GND
- J5 pad 12: TH9 -> unconnected-(J5-Pad12)
- J5 pad 13: TH8 -> unconnected-(J5-Pad13)
- J5 pad 14: TH7 -> unconnected-(J5-Pad14)
- J5 pad 15: TH6 -> unconnected-(J5-Pad15)
- J5 pad 6: unconnected-(J5-Pad6) -> TH6
- J5 pad 7: unconnected-(J5-Pad7) -> TH7
- J5 pad 8: unconnected-(J5-Pad8) -> TH8
- J5 pad 9: unconnected-(J5-Pad9) -> TH9
Routing:
- net GND: track 152.0 -> 122.9 mm
- net unconnected-(J5-Pad13): track 0.00 -> 16.2 mm
- net TH8: track 38.0 -> 21.7 mm
- net 5V: track 180.2 -> 169.3 mm
- net Net-(J1-Pin_2): track 65.7 -> 55.3 mm

Commit message: fixed?
Parts:
- moved J1 8.76 mm to (60.6, 106.2)
- moved G*** 8.40 mm to (55.2, 121.1)
Connections:
- D1 pad 1: Net-(D1-K) -> 5V
- D1 pad 2: 5V -> Net-(D1-A)
- J5 pad 10: 5V -> GND
- J5 pad 11: GND -> 5V
- J5 pad 12: unconnected-(J5-Pad12) -> TH9
- J5 pad 13: unconnected-(J5-Pad13) -> TH8
- J5 pad 14: unconnected-(J5-Pad14) -> TH7
- J5 pad 15: unconnected-(J5-Pad15) -> TH6
- J5 pad 6: TH6 -> unconnected-(J5-Pad6)
- J5 pad 7: TH7 -> unconnected-(J5-Pad7)
- J5 pad 8: TH8 -> unconnected-(J5-Pad8)
- J5 pad 9: TH9 -> unconnected-(J5-Pad9)
- K1 pad 2: Net-(D1-K) -> Net-(D1-A)
- Q1 pad 2: Net-(D1-K) -> Net-(D1-A)
Routing:
- net Net-(D1-K): track 85.7 -> 0.00 mm, vias 4 -> 0
- net TH8: track 21.7 -> 94.6 mm, vias 2 -> 4
- net Net-(D1-A): track 0.00 -> 48.7 mm, vias 0 -> 2
- net Net-(J1-Pin_2): track 55.3 -> 99.3 mm
- net 5V: track 169.3 -> 133.5 mm, vias 2 -> 4
- net GND: track 122.9 -> 105.9 mm
- net unconnected-(J5-Pad13): track 16.2 -> 0.00 mm
- net TH4: track 87.1 -> 82.2 mm
- net /24V: track 31.5 -> 35.6 mm
- net TH1: track 92.7 -> 95.2 mm
- net TH3: track 85.1 -> 82.9 mm
- net TH6: track 81.3 -> 83.3 mm, vias 0 -> 2
- net TH7: track 77.4 -> 79.0 mm, vias 0 -> 2
- net TH9: track 86.3 -> 87.8 mm, vias 2 -> 4
- net TH5: track 73.9 -> 74.9 mm, vias 1 -> 3
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
Commit message: added resistors to pcb
Parts:
- added R4: 4.7k, PCM_JLCPCB:R_1206, F.Cu at (77.7, 71.5)
- added R5: 10k, PCM_JLCPCB:R_1206, F.Cu at (103.0, 56.6)
Routing:
- net GND: track 105.9 -> 124.6 mm, vias 12 -> 11
- net 10V PWM: track 25.4 -> 29.0 mm, vias 0 -> 2
- net Net-(Q1-Pad1): track 57.1 -> 59.9 mm

Commit message: fixed a trace
Routing:
- net (no net): track 0.00 -> 15.8 mm, vias 0 -> 1

Commit message: fixed the mosfet
Routing:
- net GND: track 124.6 -> 108.5 mm, vias 11 -> 7
Changed lines of the file:
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@@
-	)
-	(segment
-		(start 114.5 65.1)
-		(end 114.5 64.1)
-		(width 1)
-		(layer "F.Cu")
-		(net 1)
 	)
 	(segment
@@
 	)
 	(segment
-		(start 114.5 65.1)
-		(end 114.5 66.9)
-		(width 1)
-		(layer "F.Cu")
-		(net 1)
-	)
-	(segment
 		(start 56.7 61.31)
 		(end 56.7 76.7)
@@
 	)
 	(segment
-		(start 114.5 65.1)
-		(end 113.1 65.1)
-		(width 1)
-		(layer "F.Cu")
-		(net 1)
-	)
-	(segment
 		(start 101.58 56.6)
 		(end 99.7 58.48)
@@
 	)
 	(segment
-		(start 115.5 66.9)
-		(end 114.5 66.9)
-		(width 1)
-		(layer "F.Cu")
-		(net 1)
-	)
-	(segment
 		(start 78.98 74.2)
 		(end 83.4 74.2)
@@
 	)
 	(segment
-		(start 114.5 66.9)
-		(end 114.5 68.3)
-		(width 1)
-		(layer "F.Cu")
-		(net 1)
-	)
-	(segment
 		(start 61.5 73.094537)
 		(end 66.705463 78.3)
@@
 	)
 	(segment
-		(start 113.1 70.8)
-		(end 113.6 71.3)
-		(width 1)
-		(layer "F.Cu")
-		(net 1)
-	)
-	(segment
 		(start 107.7 64.7)
 		(end 107.3 65.1)
@@
 	)
 	(segment
-		(start 114.5 68.3)
-		(end 115.5 68.3)
-		(width 1)
-		(layer "F.Cu")
-		(net 1)
-	)
-	(segment
-		(start 114.5 64.1)
-		(end 115.5 64.1)
-		(width 1)
-		(layer "F.Cu")
-		(net 1)
-	)
-	(segment
 		(start 99.7 62.9)
 		(end 104.1 62.9)
@@
 	)
 	(segment
-		(start 115.5 65.5)
-		(end 114.9 65.5)
-		(width 1)
-		(layer "F.Cu")
-		(net 1)
-	)
-	(segment
 		(start 66.705463 78.3)
 		(end 67.3 78.3)
@@
 	)
 	(segment
-		(start 113.1 65.1)
-		(end 113.1 70.8)
-		(width 1)
-		(layer "F.Cu")
-		(net 1)
-	)
-	(segment
 		(start 104.15 62.95)
 		(end 106.3 65.1)
@@
 	)
 	(segment
-		(start 114.9 65.5)
-		(end 114.5 65.1)
-		(width 1)
-		(layer "F.Cu")
-		(net 1)
-	)
-	(segment
 		(start 129 123)
 		(end 129.5 123.5)
@@
 	)
 	(via
-		(at 115.5 63.7)
+		(at 109.1 64.1)
 		(size 0.6)
 		(drill 0.3)
@@
 	)
 	(via
-		(at 109.1 64.1)
+		(at 113.7 57.1)
+		(size 0.6)
+		(drill 0.3)
+		(layers "F.Cu" "B.Cu")
+		(net 1)
+	)
+	(via
+		(at 67.3 78.3)
+		(size 0.6)
+		(drill 0.3)
+		(layers "F.Cu" "B.Cu")
+		(net 1)
+	)
+	(via
+		(at 107.7 64.1)
 		(size 0.6)
 		(drill 0.3)
@@
 	)
 	(via
-		(at 115.5 65.5)
-		(size 0.6)
-		(drill 0.3)
-		(layers "F.Cu" "B.Cu")
-		(free yes)
-		(net 1)
-	)
-	(via
-		(at 113.7 57.1)
-		(size 0.6)
-		(drill 0.3)
-		(layers "F.Cu" "B.Cu")
-		(net 1)
-	)
-	(via
-		(at 67.3 78.3)
-		(size 0.6)
-		(drill 0.3)
-		(layers "F.Cu" "B.Cu")
-		(net 1)
-	)
-	(via
-		(at 115.5 66.9)
-		(size 0.6)
-		(drill 0.3)
-		(layers "F.Cu" "B.Cu")
-		(free yes)
-		(net 1)
-	)
-	(via
-		(at 107.7 64.1)
-		(size 0.6)
-		(drill 0.3)
-		(layers "F.Cu" "B.Cu")
-		(free yes)
-		(net 1)
-	)
-	(via
 		(at 110.5 64.1)
 		(size 0.6)
 		(drill 0.3)
-		(layers "F.Cu" "B.Cu")
-		(free yes)
-		(net 1)
-	)
-	(via
-		(at 115.5 68.3)
-		(size 0.6)
-		(drill 0.3)

Commit message: edited sch, added footprints
Parts:
- removed C4: C47.5nf, Capacitor_SMD:C_0805_2012Metric
Routing:
- net GND: track 108.5 -> 76.9 mm, vias 7 -> 3
- net (no net): track 15.8 -> 0.00 mm, vias 1 -> 0
- net Net-(J1-Pin_2): track 99.3 -> 85.7 mm

Commit message: working on pcb
Parts:
- added C1: C4.7uf, Capacitor_SMD:C_0805_2012Metric, F.Cu at (162.0, 82.1)
- added C2: C0.1uf, Capacitor_SMD:C_0805_2012Metric, F.Cu at (103.2, 57.4)
- added C3: C4.7uf, Capacitor_SMD:C_0805_2012Metric, F.Cu at (162.0, 88.2)
- added C4: C19nf, Capacitor_SMD:C_0805_2012Metric, F.Cu at (111.0, 64.1)
- added C5: C0.1uf, Capacitor_SMD:C_0805_2012Metric, F.Cu at (162.0, 94.2)
- added C6: C0.1u, Capacitor_SMD:C_0805_2012Metric, F.Cu at (114.8, 64.1)
- added D2: V20DM100C-M3/I, Package_TO_SOT_SMD:TO-263-2, F.Cu at (88.0, 123.5)
- added R5: R0.001, CRE2512_FZ_R001E_2 (1):RESC6432X90N, F.Cu at (73.6, 110.0)
- added R6: R10, Resistor_SMD:R_0805_2012Metric, F.Cu at (107.0, 64.1)
- added R7: R1k, Resistor_SMD:R_0805_2012Metric, F.Cu at (78.2, 117.0)
- added U2: INA181, Package_TO_SOT_SMD:SOT-23-6, F.Cu at (73.3, 116.2)
- F1: value 20A Fuse -> 14 Amp Fuse
- R1, R2, R4: footprint PCM_JLCPCB:R_1206 -> Resistor_SMD:R_0805_2012Metric
- moved R5 7.65 mm to (95.4, 57.0)
- moved R3 7.31 mm to (94.8, 60.4), turned to 180 degrees
- moved MOSFET1 1.09 mm to (108.8, 72.0), turned to -90 degrees
- moved R1 0.10 mm to (121.5, 60.2)
- moved R2 0.10 mm to (121.5, 64.0)
Connections:
- F1 pad 2: Net-(F1-Pad2) -> unconnected-(F1-Pad2)
- J1 pad 2: Net-(J1-Pin_2) -> SHUNT HIGH
- J3 pad 10: unconnected-(J3-Pad10) -> Current Vout
- K1 pad 3: Net-(F1-Pad2) -> unconnected-(K1-Pad3)
- MOSFET1 pad 1: Net-(J1-Pin_2) -> GND
- MOSFET1 pad 2: Net-(J1-Pin_2) -> GND
- MOSFET1 pad 3: Net-(J1-Pin_2) -> GND
- MOSFET1 pad 4: 10V PWM -> Net-(C4-Pad1)
- MOSFET1 pad 5: GND -> HEATER OUT
- MOSFET1 pad 6: GND -> HEATER OUT
- MOSFET1 pad 7: GND -> HEATER OUT
- MOSFET1 pad 8: GND -> HEATER OUT
- Q1 pad 2: Net-(D1-A) -> GND
- Q1 pad 3: GND -> Net-(D1-A)
Routing:
- net Net-(J1-Pin_2): track 85.7 -> 0.00 mm
- net GND: track 76.9 -> 15.8 mm, vias 3 -> 2
- net 10V PWM: track 29.0 -> 0.19 mm, vias 2 -> 0
- net Net-(F1-Pad2): track 17.0 -> 0.00 mm
- net (no net): track 0.00 -> 17.0 mm
- net Net-(U1-INPUT_A): track 21.7 -> 9.94 mm
- net Net-(Q1-Pad1): track 59.9 -> 60.5 mm
- added copper zone on B.Cu, net GND
Other:
- board text removed: "TO HEATER"
